Commit message: feat(piper_description): 剪夹一体式夹爪模型替换原模型，实验可用

File: piper_ros/src/piper_description/urdf/piper_description.urdf (robot description, URDF)
Before this commit: robot piper, 11 links, 10 joints
Links:
- removed link dummy_link
- removed link gripper_base
- removed link link7
- removed link link8
- link base_link: mass 1.02 -> 0.162290652295194
- link link1: mass 0.71 -> 0.106878894462235
- link link2: mass 1.17 -> 0.203932846071332
- link link3: mass 0.5 -> 0.259293309425469
- link link4: mass 0.38 -> 0.1207071468194
- link link5: mass 0.383 -> 0.136390779513211
- link link6: mass 0.007 -> 0.297734657028244
Joints:
- removed joint base_to_dummy
- removed joint joint6_to_gripper_base
- removed joint joint7
- removed joint joint8
- joint joint1: limit lower=-2.618 upper=2.168 effort=100 velocity=5 -> lower=-2.618 upper=2.618 effort=100 velocity=5; origin xyz=0 0 0.123 rpy=0 0 0 -> xyz=0 0 0.08595 rpy=0 0 0
- joint joint2: origin xyz=0 0 0 rpy=1.5708 -0.1359 -3.1416 -> xyz=0 0.03275 0.035 rpy=1.5708 0 3.1416
- joint joint3: limit lower=-2.967 upper=0 effort=100 velocity=5 -> lower=0 upper=2.967 effort=100 velocity=5; origin xyz=0.28503 0 0 rpy=0 0 -1.7939 -> xyz=0.28358 0.028726 0 rpy=-3.1416 0 0
- joint joint4: origin xyz=-0.021984 -0.25075 0 rpy=1.5708 0 0 -> xyz=-0.21102 -0.040531 0.03275 rpy=1.5708 0 -1.4835
- joint joint5: limit lower=-1.22 upper=1.22 effort=100 velocity=5 -> lower=-1.74 upper=1.74 effort=100 velocity=5; origin xyz=0 0 0 rpy=-1.5708 0 0 -> xyz=0 0.02392 0.036 rpy=-1.5708 0 0
- joint joint6: origin xyz=8.8259E-05 -0.091 0 rpy=1.5708 0 0 -> xyz=0 -0.091 -0.02392 rpy=1.5708 0 0

Commit message: feat(collision): 新增简化模型面数 + convx hull 生成脚本，可用于减少碰撞检测计算量

File: piper_ros/src/piper_description/urdf/piper_description.urdf (robot description, URDF)
Before this commit: robot piper_description, 8 links, 7 joints
Links:
- link base_link: geometry collision mesh filename=package://piper_description/processed_meshes/visual/base_li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; visual mesh filename=package://piper_description/meshes/base_link.STL
- link link1: geometry collision mesh filename=package://piper_description/processed_meshes/visual/link1.S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; visual mesh filename=package://piper_description/meshes/link1.STL
- link link2: geometry collision mesh filename=package://piper_description/processed_meshes/visual/link2.S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; visual mesh filename=package://piper_description/meshes/link2.STL
- link link3: geometry collision mesh filename=package://piper_description/processed_meshes/visual/link3.S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; visual mesh filename=package://piper_description/meshes/link3.STL
- link link4: geometry collision mesh filename=package://piper_description/processed_meshes/visual/link4.S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; visual mesh filename=package://piper_description/meshes/link4.STL
- link link5: geometry collision mesh filename=package://piper_description/processed_meshes/visual/link5.S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; visual mesh filename=package://piper_description/meshes/link5.STL
- link link6: geometry collision mesh filename=package://piper_description/processed_meshes/visual/link6.S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; visual mesh filename=package://piper_description/meshes/link6.STL
