Commit message: feat(camera): 去掉末端的相机模型，只用真正相机的模型

File: tomato_car_description/src/tomato_car_description/urdf/tomato_car_description.urdf.xacro (robot description, xacro)
@@ -11,5 +11,5 @@
         <origin xyz="0.1124 0 0.67" rpy="0 0 0"/>
     </xacro:piper_arm>
-    <xacro:gemini335L_336L_camera prefix="wrist_cam" parent="${arm_prefix}_link6" use_collision="false">
+    <xacro:gemini335L_336L_camera prefix="wrist_cam" parent="${arm_prefix}_link6" use_collision="true">
         <origin xyz="0.041 -0.048 0.064" rpy="3.14 -1.57 0"/>
     </xacro:gemini335L_336L_camera>

File: tomato_car_description/src/tomato_car_moveit/config/gazebo_tomato_car_description.urdf (robot description, URDF)
Before this commit: robot tomato_car_description, 39 links, 38 joints
Links:
- link wrist_cam_IMU_frame: geometry collision mesh filename=package://tomato_car_description/meshes/wrist_camera/camera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; visual mesh filename=package://tomato_car_description/meshes/wrist_camera/camera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
- link wrist_cam_base_link: geometry collision mesh filename=package://tomato_car_description/meshes/wrist_camera/base_l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; visual mesh filename=package://tomato_car_description/meshes/wrist_camera/base_l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
- link wrist_cam_color_frame: geometry collision mesh filename=package://tomato_car_description/meshes/wrist_camera/camera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; visual mesh filename=package://tomato_car_description/meshes/wrist_camera/camera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
- link wrist_cam_color_optical_frame: geometry collision mesh filename=package://tomato_car_description/meshes/wrist_camera/camera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; visual mesh filename=package://tomato_car_description/meshes/wrist_camera/camera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
- link wrist_cam_color_screw_frame: geometry collision mesh filename=package://tomato_car_description/meshes/wrist_camera/camera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; visual mesh filename=package://tomato_car_description/meshes/wrist_camera/camera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
- link wrist_cam_depth_frame: geometry collision mesh filename=package://tomato_car_description/meshes/wrist_camera/camera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; visual mesh filename=package://tomato_car_description/meshes/wrist_camera/camera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
- link wrist_cam_left_ir_frame: geometry collision mesh filename=package://tomato_car_description/meshes/wrist_camera/camera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; visual mesh filename=package://tomato_car_description/meshes/wrist_camera/camera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
- link wrist_cam_left_ir_optical_frame: geometry collision mesh filename=package://tomato_car_description/meshes/wrist_camera/camera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; visual mesh filename=package://tomato_car_description/meshes/wrist_camera/camera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
- link wrist_cam_right_ir_frame: geometry collision mesh filename=package://tomato_car_description/meshes/wrist_camera/camera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; visual mesh filename=package://tomato_car_description/meshes/wrist_camera/camera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
- link wrist_cam_right_ir_optical_frame: geometry collision mesh filename=package://tomato_car_description/meshes/wrist_camera/camera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; visual mesh filename=package://tomato_car_description/meshes/wrist_camera/camera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
