Commit message: fix(car): 新增车轮 joint 临时发布节点，修正车轮关节定义 test: 测试通过，整车+机械臂+多相机+gui 整车运行，精度很高，目测精度误差小于0.25cm，再修复一个 tf 更新不及时的问题即可
Co-authored-by: Copilot <copilot@github.com>

File: tomato_car_description/src/tomato_car_description/urdf/piper_arm.xacro (robot description, xacro)
@@ -205,5 +205,5 @@
         <link name="${prefix}_link_tcp" />
         <joint name="${prefix}_joint_tcp" type="fixed">
-            <origin xyz="0 0.018 0.13181" rpy="0 0 0" />
+            <origin xyz="-0.005 0.018 0.13181" rpy="0 0 0" />
             <parent link="${prefix}_link6" />
             <child link="${prefix}_link_tcp" />

File: tomato_car_description/src/tomato_car_description/urdf/tomato_car_base.xacro (robot description, xacro)
@@ -24,5 +24,5 @@
             </collision>
         </link>
-        <link name="frot_right_wheel_link">
+        <link name="front_right_wheel_link">
             <inertial>
                 <origin xyz="7.9717E-07 -0.0031072 -4.9001E-07" rpy="0 0 0" />
@@ -33,5 +33,5 @@
                 <origin xyz="0 0 0" rpy="0 0 0" />
                 <geometry>
-                    <mesh filename="package://tomato_car_description/meshes/tomato_car/frot_right_wheel_link.STL" />
+                    <mesh filename="package://tomato_car_description/meshes/tomato_car/front_right_wheel_link.STL" />
                 </geometry>
                 <material name="">
@@ -42,16 +42,16 @@
                 <origin xyz="0 0 0" rpy="0 0 0" />
                 <geometry>
-                    <mesh filename="package://tomato_car_description/meshes/tomato_car/frot_right_wheel_link.STL" />
+                    <mesh filename="package://tomato_car_description/meshes/tomato_car/front_right_wheel_link.STL" />
                 </geometry>
             </collision>
         </link>
-        <joint name="frot_right_wheel_joint" type="revolute">
+        <joint name="front_right_wheel_joint" type="revolute">
             <origin xyz="0.6 -0.25872 -1.3111E-05" rpy="0 0 0" />
             <parent link="base_link" />
-            <child link="frot_right_wheel_link" />
+            <child link="front_right_wheel_link" />
             <axis xyz="0 0 -1" />
             <limit lower="-0.59" upper="0.59" effort="10" velocity="2"/>
         </joint>
-        <link name="frot_left_wheel_link">
+        <link name="front_left_wheel_link">
             <inertial>
                 <origin xyz="7.1211E-07 0.0035556 -6.725E-07" rpy="0 0 0" />
@@ -62,5 +62,5 @@
                 <origin xyz="0 0 0" rpy="0 0 0" />
                 <geometry>
-                    <mesh filename="package://tomato_car_description/meshes/tomato_car/frot_left_wheel_link.STL" />
+                    <mesh filename="package://tomato_car_description/meshes/tomato_car/front_left_wheel_link.STL" />
                 </geometry>
                 <material name="">
@@ -71,12 +71,12 @@
                 <origin xyz="0 0 0" rpy="0 0 0" />
                 <geometry>
-                    <mesh filename="package://tomato_car_description/meshes/tomato_car/frot_left_wheel_link.STL" />
+                    <mesh filename="package://tomato_car_description/meshes/tomato_car/front_left_wheel_link.STL" />
                 </geometry>
             </collision>
         </link>
-        <joint name="frot_left_wheel_joint" type="revolute">
+        <joint name="front_left_wheel_joint" type="revolute">
             <origin xyz="0.6 0.25872 -1.3105E-05" rpy="0 0 0" />
             <parent link="base_link" />
-            <child link="frot_left_wheel_link" />
+            <child link="front_left_wheel_link" />
             <axis xyz="0 0 1" />
             <limit lower="-0.59" upper="0.59" effort="10" velocity="2"/>

File: tomato_car_description/src/tomato_car_moveit/config/gazebo_tomato_car_description.urdf (robot description, URDF)
Before this commit: robot tomato_car_description, 39 links, 38 joints
Links:
- removed link frot_left_wheel_link
- removed link frot_right_wheel_link
- added link front_left_wheel_link, mass 1.4097; collision mesh filename=package://tomato_car_description/meshes/tomato_car/front_le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; visual mesh filename=package://tomato_car_description/meshes/tomato_car/front_le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
- added link front_right_wheel_link, mass 1.4097; collision mesh filename=package://tomato_car_description/meshes/tomato_car/front_ri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; visual mesh filename=package://tomato_car_description/meshes/tomato_car/front_ri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
Joints:
- removed joint frot_left_wheel_joint
- removed joint frot_right_wheel_joint
- added joint front_left_wheel_joint: type revolute, parent base_link, child front_left_wheel_link, origin xyz=0.6 0.25872 -1.3105E-05 rpy=0 0 0, axis 0 0 1, limit lower=-0.59 upper=0.59 effort=10 velocity=2
- added joint front_right_wheel_joint: type revolute, parent base_link, child front_right_wheel_link, origin xyz=0.6 -0.25872 -1.3111E-05 rpy=0 0 0, axis 0 0 -1, limit lower=-0.59 upper=0.59 effort=10 velocity=2
